File: fmc_esdi_drive/fmc_esdi_drive.kicad_pcb (KiCad board)
At the start: 2 copper layers, 98 x 59.7 mm, 37 parts, among them J1 ASP-134604-01, J2 Control Cable, J3 Data Port A, J4 Data Port B, U1 MAX17501BxTB, U10 74LS06, U6 74LS06, U7 74LS06

Commit message: Finish FMC adapter PCB
Parts:
- added C10: C, Capacitor_SMD:C_0402_1005Metric, F.Cu at (231.8, 134.0)
- added C11: C, Capacitor_SMD:C_0402_1005Metric, F.Cu at (243.1, 130.6)
- added C12: C, Capacitor_SMD:C_0402_1005Metric, F.Cu at (222.5, 122.9)
- added C13: C, Capacitor_SMD:C_0402_1005Metric, F.Cu at (232.7, 122.9)
- added C14: C, Capacitor_SMD:C_0402_1005Metric, F.Cu at (242.8, 122.9)
- added C15: C, Capacitor_SMD:C_0402_1005Metric, F.Cu at (253.0, 122.9)
- added C16: C, Capacitor_SMD:C_0402_1005Metric, F.Cu at (263.1, 122.9)
- added C17: C, Capacitor_SMD:C_0402_1005Metric, F.Cu at (273.3, 122.9)
- added C5: C, Capacitor_SMD:C_0402_1005Metric, F.Cu at (188.5, 123.4)
- added C6: C, Capacitor_SMD:C_0402_1005Metric, F.Cu at (196.1, 123.4)
- added C7: C, Capacitor_SMD:C_0402_1005Metric, F.Cu at (203.7, 123.4)
- added C8: C, Capacitor_SMD:C_0402_1005Metric, F.Cu at (211.3, 123.4)
- added C9: C, Capacitor_SMD:C_0402_1005Metric, F.Cu at (221.6, 134.0)
- moved R7 17.8 mm to (209.0, 132.1), turned to 180 degrees
- moved U13 15.9 mm to (207.8, 127.0)
- moved U14 14.8 mm to (200.2, 127.0)
- moved U9 13.4 mm to (184.9, 127.0)
- moved R8 13.1 mm to (201.4, 132.1), turned to 180 degrees
- moved U8 12.2 mm to (192.5, 127.0)
- moved C1 11.1 mm to (268.7, 132.6), turned to 0 degrees
- moved JP2 11.0 mm to (252.7, 137.2), turned to 180 degrees
- moved R1 11.0 mm to (260.5, 131.6)
- moved U1 10.7 mm to (265.9, 136.3), turned to -90 degrees
- moved C3 9.49 mm to (264.4, 132.0)
- moved R4 8.06 mm to (186.2, 132.1), turned to 180 degrees
- moved R2 6.06 mm to (260.5, 135.6)
- moved L1 5.88 mm to (271.0, 139.8), turned to 0 degrees
- moved C4 5.77 mm to (270.3, 135.2), turned to 180 degrees
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Connections:
- J1 pad G18: WRITE_DATA_A_FMC -> WRITE_CLOCK_A_FMC
- J1 pad G21: WRITE_DATA_B_FMC -> WRITE_CLOCK_B_FMC
- J1 pad G30: DRIVE_SELECTED_B_FMC -> INDEX_UNGATED_B_FMC
- J1 pad G31: CMD_COMPLETE_B_FMC -> SECTOR_UNGATED_B_FMC
- J1 pad G33: READ_CLOCK_A_FMC -> READ_DATA_A_FMC
- J1 pad G36: READ_CLOCK_B_FMC -> READ_DATA_B_FMC
- J1 pad H16: WRITE_CLOCK_A_FMC -> WRITE_DATA_A_FMC
- J1 pad H19: WRITE_CLOCK_B_FMC -> WRITE_DATA_B_FMC
- J1 pad H31: SECTOR_UNGATED_B_FMC -> DRIVE_SELECTED_B_FMC
- J1 pad H32: INDEX_UNGATED_B_FMC -> CMD_COMPLETE_B_FMC
- J1 pad H34: READ_DATA_A_FMC -> READ_CLOCK_A_FMC
- J1 pad H37: READ_DATA_B_FMC -> READ_CLOCK_B_FMC
- RN1 pad 2: HEAD3 -> HEAD2
- RN1 pad 3: HEAD2 -> HEAD0
- RN1 pad 4: WRITE_GATE -> XFER_REQ
- RN1 pad 5: HEAD0 -> DRIVE0
- RN1 pad 6: HEAD1 -> DRIVE1
- RN1 pad 7: XFER_REQ -> DRIVE2
- RN1 pad 8: DRIVE0 -> READ_GATE
- RN1 pad 9: DRIVE1 -> CMD_DATA
- RN2 pad 2: DRIVE2 -> HEAD3
- RN2 pad 3: READ_GATE -> WRITE_GATE
- RN2 pad 4: CMD_DATA -> HEAD1
- U10 pad 1: Net-(U3-B5) -> SECTOR_UNGATED_B_5V
- U10 pad 12: unconnected-(U10-Pad12) -> CMD_COMPLETE_B
- U10 pad 13: GND -> CMD_COMPLETE_B_5V
- U10 pad 2: CMD_COMPLETE_B -> SECTOR_UNGATED_B
- U10 pad 3: Net-(U3-B6) -> GND
- U10 pad 4: INDEX_UNGATED_B -> unconnected-(U10-Pad4)
- U11 pad 16: unconnected-(U11-B6-Pad16) -> Net-(U11-B6)
- U11 pad 17: unconnected-(U11-B5-Pad17) -> Net-(U11-B5)
- U11 pad 20: Net-(U11-B2) -> CMD_COMPLETE_B_5V
- U11 pad 21: Net-(U11-B1) -> SECTOR_UNGATED_B_5V
- U11 pad 3: READ_CLOCK_A_FMC -> SECTOR_UNGATED_B_FMC
- U11 pad 4: READ_DATA_A_FMC -> CMD_COMPLETE_B_FMC
- U11 pad 5: READ_CLOCK_B_FMC -> READ_DATA_A_FMC
- U11 pad 6: READ_DATA_B_FMC -> READ_CLOCK_A_FMC
- U11 pad 7: GND -> READ_DATA_B_FMC
- U11 pad 8: GND -> READ_CLOCK_B_FMC
- U12 pad 3: WRITE_CLOCK_A_FMC -> WRITE_DATA_A_FMC
- U12 pad 4: WRITE_DATA_A_FMC -> WRITE_CLOCK_A_FMC
- U12 pad 5: WRITE_CLOCK_B_FMC -> WRITE_DATA_B_FMC
- U12 pad 6: WRITE_DATA_B_FMC -> WRITE_CLOCK_B_FMC
- U13 pad 2: Net-(U12-B3) -> Net-(U12-B4)
- U13 pad 3: Net-(U11-B3) -> Net-(U11-B6)
- U14 pad 2: Net-(U12-B4) -> Net-(U12-B3)
- U14 pad 3: Net-(U11-B4) -> Net-(U11-B5)
- U2 pad 10: SECTOR_UNGATED_A_FMC -> GND
- U2 pad 14: Net-(U2-B8) -> unconnected-(U2-B8-Pad14)
- U2 pad 15: Net-(U2-B7) -> unconnected-(U2-B7-Pad15)
- U2 pad 9: DRIVE_SELECTED_A_FMC -> GND
- U3 pad 3: CMD_COMPLETE_A_FMC -> DRIVE_SELECTED_A_FMC
- U3 pad 4: INDEX_UNGATED_A_FMC -> SECTOR_UNGATED_A_FMC
- U3 pad 5: DRIVE_SELECTED_B_FMC -> CMD_COMPLETE_A_FMC
- U3 pad 6: SECTOR_UNGATED_B_FMC -> INDEX_UNGATED_A_FMC
- U3 pad 7: CMD_COMPLETE_B_FMC -> INDEX_UNGATED_B_FMC
- U3 pad 8: INDEX_UNGATED_B_FMC -> DRIVE_SELECTED_B_FMC
- U6 pad 10: INDEX_GATED -> SECTOR_GATED
- U6 pad 11: Net-(U2-B5) -> Net-(U2-B4)
- U6 pad 12: READY -> XFER_ACK
- U6 pad 13: Net-(U2-B6) -> Net-(U2-B2)
- U6 pad 3: Net-(U2-B2) -> Net-(U2-B3)
- U6 pad 4: XFER_ACK -> ATTN
- U6 pad 5: Net-(U2-B3) -> Net-(U2-B5)
- U6 pad 6: ATTN -> INDEX_GATED
- U6 pad 8: SECTOR_GATED -> READY
- U6 pad 9: Net-(U2-B4) -> Net-(U2-B6)
- U7 pad 1: Net-(U2-B7) -> Net-(U3-B1)
- U7 pad 10: DRIVE_SELECTED_B -> INDEX_UNGATED_A
- U7 pad 11: Net-(U3-B3) -> Net-(U3-B4)
- U7 pad 12: SECTOR_UNGATED_B -> SECTOR_UNGATED_A
- U7 pad 13: Net-(U3-B4) -> Net-(U3-B2)
- U7 pad 3: Net-(U2-B8) -> Net-(U3-B3)
- U7 pad 4: SECTOR_UNGATED_A -> CMD_COMPLETE_A
- U7 pad 5: Net-(U3-B1) -> Net-(U3-B5)
- U7 pad 6: CMD_COMPLETE_A -> INDEX_UNGATED_B
- U7 pad 8: INDEX_UNGATED_A -> DRIVE_SELECTED_B
- U7 pad 9: Net-(U3-B2) -> Net-(U3-B6)
- U8 pad 2: Net-(U12-B1) -> Net-(U12-B2)
- U8 pad 3: Net-(U11-B1) -> Net-(U11-B4)
- U9 pad 2: Net-(U12-B2) -> Net-(U12-B1)
- U9 pad 3: Net-(U11-B2) -> Net-(U11-B3)
Routing:
- net FMC_12V: track 0.00 -> 104.7 mm
- net FMC_VADJ: track 0.00 -> 76.1 mm, vias 0 -> 7
- net CONFIG_STAT_DATA: track 0.00 -> 71.7 mm, vias 0 -> 1
- net AME_A: track 0.00 -> 71.7 mm, vias 0 -> 3
- net Net-(U12-B1): track 0.00 -> 69.2 mm, vias 0 -> 2
- net HEAD2: track 0.00 -> 67.3 mm
- net HEAD3: track 0.00 -> 67.2 mm
- net ATTN: track 0.00 -> 65.4 mm, vias 0 -> 1
- net WRITE_GATE: track 0.00 -> 65.3 mm
- net XFER_ACK: track 0.00 -> 64.2 mm, vias 0 -> 1
- net AME_B: track 0.00 -> 60.5 mm, vias 0 -> 2
- net Net-(U12-B2): track 0.00 -> 59.8 mm, vias 0 -> 2
- net HEAD0: track 0.00 -> 57.3 mm
- net SECTOR_GATED: track 0.00 -> 55.1 mm, vias 0 -> 1
- net INDEX_UNGATED_A: track 0.00 -> 54.1 mm, vias 0 -> 1
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- added copper zone on B.Cu, net +5V
- added copper zone on F.Cu, net +5V
- added copper zone on B.Cu, net GND
- added copper zone on F.Cu, net GND
Other:
- outline, holes or cut-outs redrawn
