File: fmc_esdi_drive/oc_outputs.kicad_sch (KiCad schematic)
At the start: 5 parts, among them U10 74LS06, U6 74LS06, U7 74LS06

Commit message: PCB: Add hopeful board outline
Parts:
- U10, U6, U7: footprint (none) -> Package_SO:SOIC-14_3.9x8.7mm_P1.27mm
- U2, U3: footprint (none) -> Package_SO:TSSOP-24_4.4x7.8mm_P0.65mm
Changed lines of the file:
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@@
       (effects (font (size 1.27 1.27)))
     )
-    (property "Footprint" "" (at 99.06 82.55 0)
+    (property "Footprint" "Package_SO:SOIC-14_3.9x8.7mm_P1.27mm" (at 99.06 82.55 0)
       (effects (font (size 1.27 1.27)) hide)
     )
@@
       (effects (font (size 1.27 1.27)) (justify left))
     )
-    (property "Footprint" "" (at 48.26 175.26 0)
+    (property "Footprint" "Package_SO:SOIC-14_3.9x8.7mm_P1.27mm" (at 48.26 175.26 0)
       (effects (font (size 1.27 1.27)) hide)
     )
@@
       (effects (font (size 1.27 1.27)))
     )
-    (property "Footprint" "" (at 99.06 113.03 0)
+    (property "Footprint" "Package_SO:SOIC-14_3.9x8.7mm_P1.27mm" (at 99.06 113.03 0)
       (effects (font (size 1.27 1.27)) hide)
     )
@@
       (effects (font (size 1.27 1.27)))
     )
-    (property "Footprint" "" (at 104.14 74.93 0)
+    (property "Footprint" "Package_SO:SOIC-14_3.9x8.7mm_P1.27mm" (at 104.14 74.93 0)
       (effects (font (size 1.27 1.27)) hide)
     )
@@
       (effects (font (size 1.27 1.27)))
     )
-    (property "Footprint" "" (at 104.14 90.17 0)
+    (property "Footprint" "Package_SO:SOIC-14_3.9x8.7mm_P1.27mm" (at 104.14 90.17 0)
       (effects (font (size 1.27 1.27)) hide)
     )
@@
       (effects (font (size 1.27 1.27)))
     )
-    (property "Footprint" "" (at 114.3 168.91 0)
+    (property "Footprint" "Package_SO:SOIC-14_3.9x8.7mm_P1.27mm" (at 114.3 168.91 0)
       (effects (font (size 1.27 1.27)) hide)
     )
@@
       (effects (font (size 1.27 1.27)) (justify left))
     )
-    (property "Footprint" "" (at 69.85 175.26 0)
+    (property "Footprint" "Package_SO:SOIC-14_3.9x8.7mm_P1.27mm" (at 69.85 175.26 0)
       (effects (font (size 1.27 1.27)) hide)
     )
@@
       (effects (font (size 1.27 1.27)))
     )
-    (property "Footprint" "" (at 114.3 184.15 0)
+    (property "Footprint" "Package_SO:SOIC-14_3.9x8.7mm_P1.27mm" (at 114.3 184.15 0)
       (effects (font (size 1.27 1.27)) hide)
     )
@@
       (effects (font (size 1.27 1.27)))
     )
-    (property "Footprint" "" (at 64.77 73.66 0)
+    (property "Footprint" "Package_SO:TSSOP-24_4.4x7.8mm_P0.65mm" (at 64.77 73.66 0)
       (effects (font (size 1.27 1.27)) hide)
     )
@@
       (effects (font (size 1.27 1.27)))
     )
-    (property "Footprint" "" (at 139.7 184.15 0)
+    (property "Footprint" "Package_SO:SOIC-14_3.9x8.7mm_P1.27mm" (at 139.7 184.15 0)
       (effects (font (size 1.27 1.27)) hide)
     )
@@
       (effects (font (size 1.27 1.27)))
     )
-    (property "Footprint" "" (at 231.775 105.41 0)
+    (property "Footprint" "Package_SO:SOIC-14_3.9x8.7mm_P1.27mm" (at 231.775 105.41 0)
       (effects (font (size 1.27 1.27)) hide)
     )
@@
       (effects (font (size 1.27 1.27)))
     )
-    (property "Footprint" "" (at 226.695 82.55 0)
+    (property "Footprint" "Package_SO:SOIC-14_3.9x8.7mm_P1.27mm" (at 226.695 82.55 0)
       (effects (font (size 1.27 1.27)) hide)
     )
@@
       (effects (font (size 1.27 1.27)))
     )
-    (property "Footprint" "" (at 231.775 74.93 0)
+    (property "Footprint" "Package_SO:SOIC-14_3.9x8.7mm_P1.27mm" (at 231.775 74.93 0)
       (effects (font (size 1.27 1.27)) hide)
     )
@@
       (effects (font (size 1.27 1.27)))
     )
-    (property "Footprint" "" (at 226.695 67.31 0)
+    (property "Footprint" "Package_SO:SOIC-14_3.9x8.7mm_P1.27mm" (at 226.695 67.31 0)
       (effects (font (size 1.27 1.27)) hide)
     )
@@
       (effects (font (size 1.27 1.27)))
     )
-    (property "Footprint" "" (at 104.14 120.65 0)
+    (property "Footprint" "Package_SO:SOIC-14_3.9x8.7mm_P1.27mm" (at 104.14 120.65 0)
       (effects (font (size 1.27 1.27)) hide)
     )
@@
       (effects (font (size 1.27 1.27)))
     )
-    (property "Footprint" "" (at 139.7 168.91 0)
+    (property "Footprint" "Package_SO:SOIC-14_3.9x8.7mm_P1.27mm" (at 139.7 168.91 0)
       (effects (font (size 1.27 1.27)) hide)
     )
@@
       (effects (font (size 1.27 1.27)) (justify left))
     )
-    (property "Footprint" "" (at 26.67 175.26 0)
+    (property "Footprint" "Package_SO:SOIC-14_3.9x8.7mm_P1.27mm" (at 26.67 175.26 0)
       (effects (font (size 1.27 1.27)) hide)
     )
@@
       (effects (font (size 1.27 1.27)))
     )
-    (property "Footprint" "" (at 226.695 97.79 0)
+    (property "Footprint" "Package_SO:SOIC-14_3.9x8.7mm_P1.27mm" (at 226.695 97.79 0)
       (effects (font (size 1.27 1.27)) hide)
     )
@@
       (effects (font (size 1.27 1.27)))
     )
-    (property "Footprint" "" (at 231.775 90.17 0)
+    (property "Footprint" "Package_SO:SOIC-14_3.9x8.7mm_P1.27mm" (at 231.775 90.17 0)
       (effects (font (size 1.27 1.27)) hide)
     )
@@
       (effects (font (size 1.27 1.27)))
     )
-    (property "Footprint" "" (at 104.14 105.41 0)
+    (property "Footprint" "Package_SO:SOIC-14_3.9x8.7mm_P1.27mm" (at 104.14 105.41 0)
       (effects (font (size 1.27 1.27)) hide)
     )
@@
       (effects (font (size 1.27 1.27)))
     )
-    (property "Footprint" "" (at 99.06 67.31 0)
+    (property "Footprint" "Package_SO:SOIC-14_3.9x8.7mm_P1.27mm" (at 99.06 67.31 0)
       (effects (font (size 1.27 1.27)) hide)
     )
@@
       (effects (font (size 1.27 1.27)))
     )
-    (property "Footprint" "" (at 192.405 73.66 0)
+    (property "Footprint" "Package_SO:TSSOP-24_4.4x7.8mm_P0.65mm" (at 192.405 73.66 0)
       (effects (font (size 1.27 1.27)) hide)
     )
@@
       (effects (font (size 1.27 1.27)))
     )
-    (property "Footprint" "" (at 99.06 97.79 0)
-      (effects (font (size 1.27 1.27)) hide)
-    )
+    (property "Footprint" "Package_SO:SOIC-14_3.9x8.7mm_P1.27mm" (at 99.06 97.79 0)
+      (effects (font (size 1.27 1.27)) hide)
+    )

Commit message: Finish FMC adapter PCB
Parts:
- added C11, C12, C13, C14, C15: C, Capacitor_SMD:C_0402_1005Metric, symbol Device:C
Connections:
- net CMD_COMPLETE_B_FMC is gone; now on net INDEX_UNGATED_B_FMC: U3.7 (A5)
- net SECTOR_UNGATED_B_FMC is gone; now on net INDEX_UNGATED_A_FMC: U3.6 (A4)
- net +5V: now also C11.1, C12.1, C13.1, C14.1, C15.1
- net ATTN: now also U6.4; no longer U6.6
- net CMD_COMPLETE_A: now also U7.4; no longer U7.6
- net CMD_COMPLETE_A_FMC: now also U3.5 (A3); no longer U3.3 (A1)
- net CMD_COMPLETE_B: now also U10.12; no longer U10.2
- net DRIVE_SELECTED_A_FMC: now also U3.3 (A1); no longer U2.9 (A7)
- net DRIVE_SELECTED_B: now also U7.8; no longer U7.10
- net DRIVE_SELECTED_B_FMC: now also U3.8 (A6); no longer U3.5 (A3)
- net GND: now also U10.3, U2.10 (A8), U2.9 (A7), C11.2, C12.2, C13.2, C14.2, C15.2; no longer U10.13
- net INDEX_GATED: now also U6.6; no longer U6.10
- net INDEX_UNGATED_A: now also U7.10; no longer U7.8
- net INDEX_UNGATED_A_FMC: no longer U3.4 (A2)
- net INDEX_UNGATED_B: now also U7.6; no longer U10.4
- net INDEX_UNGATED_B_FMC: no longer U3.8 (A6)
- net READY: now also U6.8; no longer U6.12
- net SECTOR_GATED: now also U6.10; no longer U6.8
- net SECTOR_UNGATED_A: now also U7.12; no longer U7.4
- net SECTOR_UNGATED_A_FMC: now also U3.4 (A2); no longer U2.10 (A8)
- net SECTOR_UNGATED_B: now also U10.2; no longer U7.12
- net XFER_ACK: now also U6.12; no longer U6.4
- net at U6.5: now also U2.17 (B5); no longer U2.19 (B3)
- net at U7.1: now also U3.21 (B1); no longer U2.15 (B7)
- net at U6.3: now also U2.19 (B3); no longer U2.20 (B2)
- net at U6.9: now also U2.16 (B6); no longer U2.18 (B4)
- net at U2.14 (B8): no longer U7.3
- net at U6.13: now also U2.20 (B2); no longer U2.16 (B6)
- net at U6.11: now also U2.18 (B4); no longer U2.17 (B5)
- net at U3.16 (B6): now also U7.9; no longer U10.3
- net at U7.11: now also U3.18 (B4); no longer U3.19 (B3)
- net at U3.20 (B2): now also U7.13; no longer U7.9
- net at U7.5: now also U3.17 (B5); no longer U3.21 (B1)
- net SECTOR_UNGATED_B_5V: now reaches U10.1
- net SECTOR_UNGATED_B_5V: no longer U3.17 (B5)
- new net: U3.19 (B3), U7.3
- new net CMD_COMPLETE_B_5V: U10.13
- no-connect marks 6 -> 8
Other:
- moved on the sheet: U10A, U10B, U10E, U10F, U3, U6B, U6C, U6D, U6E, U6F, U7A, U7B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
